File: Kevin Splitflap/PCBs/Kicad/SplitFlapDriverV5.kicad_pcb.kicad_sch (KiCad schematic)
At the start: 25 parts, among them J1 UPDI Programming, J2 Conn_01x01_Pin, J3 Stepper Connector, J4 Hall Effect, J5 Conn_01x05_Pin, J6 Conn_01x01_Pin, J7 Conn_01x01_Pin, J8 Conn_01x01_Pin, U1 ATtiny1616-MNR, U2 ULN2003ADR, U3 SN65HVD72DR, U5 SPX3819M5-L-3-3, U6 SPX3819M5-L-5-0

Commit message: Add driver board V5 and update the BOM
Driver board V5 replaces V4 in PCBs/Kicad:
- RS-485 on the ATtiny1616 hardware USART (TXD PA1, RXD PA2, DE/RE PA4)
- Narrow 3.9 mm SOIC footprints for U2 (ULN2003ADR) and U3 (SN65HVD72DR)
- Polyfuse F1 and reverse-polarity Schottky D3 on the 12 V input
- R3 DE/RE pull-down, R4 RXD pull-up, C10/C11 decoupling
- JLCPCB part numbers on every placed part; headers and pogo pads DNP
- JLCPCB production files (Gerbers, BOM, CPL)

BOM.md: V5 parts table and the actual JLCPCB checkout total
($327.23 for 50 boards incl. customs and shipping), with updated totals.

Also adds the proposal .docx source.
Parts:
- removed R1: 0R, Resistor_SMD:R_0805_2012Metric, symbol Device:R
- added C10, C11: 100nF, Capacitor_SMD:C_0603_1608Metric, symbol Device:C
- added D3: D_Schottky, Diode_SMD:D_SMA, symbol Device:D_Schottky
- added F1: 750mA/24V, Fuse:Fuse_1812_4532Metric, symbol Device:Polyfuse_Small
- added R3, R4: 10k, Resistor_SMD:R_0603_1608Metric, symbol Device:R
- C1: footprint Capacitor_SMD:C_Elec_5x5.4 -> Capacitor_SMD:CP_Elec_6.3x5.4; FT Rotation Offset (none) -> 180; JLCPCB Part Number (none) -> C4747964
- C2, C3, C6, C8: JLCPCB Part Number (none) -> C1623
- C4: footprint Capacitor_SMD:C_0603_1608Metric -> Capacitor_SMD:C_0805_2012Metric; JLCPCB Part Number (none) -> C15850
- C5, C9: JLCPCB Part Number (none) -> C19702
- C7: value 100n -> 100nF; JLCPCB Part Number (none) -> C14663
- D1: JLCPCB Part Number (none) -> C2286
- J1, J2, J5, J6, J7, J8: now not fitted
- J3: FT Rotation Offset (none) -> 180; JLCPCB Part Number (none) -> C157991
- J4: FT Rotation Offset (none) -> 180; JLCPCB Part Number (none) -> C131339
- R2: value 60R -> 470R; JLCPCB Part Number (none) -> C23179
- U1: FT Rotation Offset (none) -> 270
- U2: footprint Package_SO:SOIC-16W_5.3x10.2mm_P1.27mm -> Package_SO:SOIC-16_3.9x9.9mm_P1.27mm
- U3: footprint Package_SO:SOIC-8_5.3x6.2mm_P1.27mm -> Package_SO:SOIC-8_3.9x4.9mm_P1.27mm
- U5: FT Rotation Offset (none) -> 90; JLCPCB Part Number (none) -> C9055
- U6: FT Rotation Offset (none) -> 90; JLCPCB Part Number (none) -> C13417
Connections:
- net +3V3: now also C10.1, C11.1, R4.1
- net +VBUS: now also F1.2; no longer C2.1
- net +VBUSF: now also D3.1 (K)
- net DE/RE: now also U1.5 (PA4), R3.1; no longer U1.7 (PA6)
- net GND: now also C10.2, C11.2, R3.2
- net IO1: now also U1.8 (PA7); no longer U1.1 (PA2)
- net IO2: now also U1.6 (PA5); no longer U1.20 (PA1)
- net RXD: now also U1.1 (PA2), R4.2; no longer U1.8 (PA7)
- net TXD: now also U1.20 (PA1); no longer U1.6 (PA5)
- new net: C2.1, D3.2 (A), F1.1
- no-connect marks 0 -> 9
Other:
- moved on the sheet: U3
