File: Kevin Splitflap/PCBs/Driverv5/SplitFlapDriverV5.kicad_pcb.kicad_pcb (KiCad board)
At the start: 2 copper layers, 30 x 60 mm, 30 parts, among them J1 UPDI Programming, J2 Conn_01x01_Pin, J3 Stepper Connector, J4 Hall Effect, J5 Conn_01x05_Pin, J6 Conn_01x01_Pin, J7 Conn_01x01_Pin, J8 Conn_01x01_Pin, U1 ATtiny1616-MNR, U2 ULN2003ADR, U3 SN65HVD72DR, U5 SPX3819M5-L-3-3, U6 SPX3819M5-L-5-0

Commit message: Add bus boards, ground PC0 on driver V5, update BOM totals
- Move the driver V5 KiCad project from PCBs/Kicad to PCBs/Driverv5 and
  tie PC0 to GND as a board ID; production files regenerated.
- Add PCBs/bus-board-5-module: Adam G's 202 mm 5-module bus board rebuilt
  in KiCad with the A/B labels corrected to match the driver board.
- Add PCBs/bus-board: single-piece 606 mm bus board for a 15-module row
  (not ordered).
- BOM: bus boards ordered with the driver boards (JLCPCB checkout $348.75
  for both); wall total now ~$774.53, grand total ~$993.
- Add Driverv5.zip snapshot.
Connections:
- U1 pad 15: unconnected-(U1-PC0-Pad15) -> GND
Routing:
- net GND: track 29.8 -> 31.1 mm, vias 19 -> 20
Changed lines of the file:
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@@
 			(size 0.143431 0.143431)
 			(layers "F.Cu" "F.Mask" "F.Paste")
-			(net "unconnected-(U1-PC0-Pad15)")
+			(net "GND")
 			(pinfunction "PC0_15")
-			(pintype "bidirectional+no_connect")
+			(pintype "bidirectional")
 			(options
 				(clearance outline)
@@
 	)
 	(segment
+		(start 139.4 96.25)
+		(end 139.4 96.4)
+		(width 0.2)
+		(layer "F.Cu")
+		(net "GND")
+	)
+	(segment
 		(start 142.925 88.025)
 		(end 143.6 87.35)
@@
 	)
 	(segment
+		(start 139.4 96.4)
+		(end 140.2 97.2)
+		(width 0.2)
+		(layer "F.Cu")
+		(net "GND")
+	)
+	(segment
 		(start 126.25 104.7)
 		(end 126.25 103.55)
@@
 		(net "GND")
 	)
+	(via
+		(at 140.2 97.2)
+		(size 0.6)
+		(drill 0.3)
+		(layers "F.Cu" "B.Cu")
+		(net "GND")
+	)

Commit message: Driver V5: swap U3 to THVD1400DR, update BOM costs
THVD1400DR (C3235232) is a drop-in for the SN65HVD72DR in the same
SOIC-8 pinout: 3-5.5 V, 500 kbps, failsafe, 1/8 unit load, +/-16 V bus
fault protection, at about a quarter of the price. No layout or firmware
change. BOM totals adjusted by ~$68 pending a JLC re-quote.
Parts:
- U3: value SN65HVD72DR -> THVD1400DR
Changed lines of the file:
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@@
 			)
 		)
-		(property "Value" "SN65HVD72DR"
+		(property "Value" "THVD1400DR"
 			(at 2.375 3.4 0)
 			(layer "F.Fab")
@@
 			)
 		)
-		(property "Datasheet" "http://www.ti.com/lit/ds/symlink/sn65hvd11-ht.pdf"
+		(property "Datasheet" "https://www.ti.com/lit/ds/symlink/thvd1400.pdf"
 			(at 0 0 0)
 			(layer "F.Fab")
@@
 			)
 		)
-		(property "Description" "3.3V, RS-485 Transceiver, SOIC-8"
+		(property "Description" "3-5.5V, 500kbps RS-485 Transceiver, SOIC-8"
 			(at 0 0 0)
 			(layer "F.Fab")
@@
 			)
 		)
-		(property "Manufacturer Part Number" "SN65HVD72DR"
+		(property "Manufacturer Part Number" "THVD1400DR"
 			(at 0 0 180)
 			(unlocked yes)
@@
 			)
 		)
-		(property "JLCPCB Part Number" "C48125"
+		(property "JLCPCB Part Number" "C3235232"
 			(at 0 0 180)
 			(unlocked yes)
