File: Kevin Splitflap/PCBs/Driverv5/SplitFlapDriverV5.kicad_pcb.kicad_sch (KiCad schematic)
At the start: 30 parts, among them J1 UPDI Programming, J2 Conn_01x01_Pin, J3 Stepper Connector, J4 Hall Effect, J5 Conn_01x05_Pin, J6 Conn_01x01_Pin, J7 Conn_01x01_Pin, J8 Conn_01x01_Pin, U1 ATtiny1616-MNR, U2 ULN2003ADR, U3 SN65HVD72DR, U5 SPX3819M5-L-3-3, U6 SPX3819M5-L-5-0

Commit message: Add bus boards, ground PC0 on driver V5, update BOM totals
- Move the driver V5 KiCad project from PCBs/Kicad to PCBs/Driverv5 and
  tie PC0 to GND as a board ID; production files regenerated.
- Add PCBs/bus-board-5-module: Adam G's 202 mm 5-module bus board rebuilt
  in KiCad with the A/B labels corrected to match the driver board.
- Add PCBs/bus-board: single-piece 606 mm bus board for a 15-module row
  (not ordered).
- BOM: bus boards ordered with the driver boards (JLCPCB checkout $348.75
  for both); wall total now ~$774.53, grand total ~$993.
- Add Driverv5.zip snapshot.
Connections:
- net GND: now also U1.15 (PC0)
- no-connect marks 9 -> 8
Changed lines of the file:
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@@
-	)
-	(no_connect
-		(at 38.1 77.47)
 	)
 	(no_connect
@@
 		(pts
 			(xy 34.29 80.01) (xy 38.1 80.01)
+		)
+		(stroke
+			(width 0)
+			(type default)
+		)
+	)
+	(wire
+		(pts
+			(xy 33.02 77.47) (xy 38.1 77.47)
 		)
 		(stroke
@@
 					(unit 1)
 				)
+			)
+		)
+	)
+	(symbol
+		(lib_id "power:GND")
+		(at 33.02 77.47 270)
+		(unit 1)
+		(body_style 1)
+		(exclude_from_sim no)
+		(in_bom yes)
+		(on_board yes)
+		(in_pos_files yes)
+		(dnp no)
+		(fields_autoplaced yes)
+		(property "Reference" "#PWR033"
+			(at 26.67 77.47 0)
+			(hide yes)
+			(show_name no)
+			(do_not_autoplace no)
+			(effects
+				(font
+					(size 1.27 1.27)
+				)
+			)
+		)
+		(property "Value" "GND"
+			(at 29.21 77.4699 90)
+			(show_name no)
+			(do_not_autoplace no)
+			(effects
+				(font
+					(size 1.27 1.27)
+				)
+				(justify right)
+			)
+		)
+		(property "Footprint" ""
+			(at 33.02 77.47 0)
+			(hide yes)
+			(show_name no)
+			(do_not_autoplace no)
+			(effects
+				(font
+					(size 1.27 1.27)
+				)
+			)
+		)
+		(property "Datasheet" ""
+			(at 33.02 77.47 0)
+			(hide yes)
+			(show_name no)
+			(do_not_autoplace no)
+			(effects
+				(font
+					(size 1.27 1.27)
+				)
+			)
+		)
+		(property "Description" "Power symbol creates a global label with name \"GND\" , ground"
+			(at 33.02 77.47 0)
+			(hide yes)
+			(show_name no)
+			(do_not_autoplace no)
+			(effects
+				(font
+					(size 1.27 1.27)
+				)
+			)
+		)
+		(pin "1"
+		)
+		(instances
+			(project "SplitFlapDriverV5.kicad_pcb"
+				(path "/2dad463d-4b58-4df7-9a4a-fb5d7d6b5e7d"
+					(reference "#PWR033")
+					(unit 1)
+				)

Commit message: Driver V5: swap U3 to THVD1400DR, update BOM costs
THVD1400DR (C3235232) is a drop-in for the SN65HVD72DR in the same
SOIC-8 pinout: 3-5.5 V, 500 kbps, failsafe, 1/8 unit load, +/-16 V bus
fault protection, at about a quarter of the price. No layout or firmware
change. BOM totals adjusted by ~$68 pending a JLC re-quote.
Parts:
- U3: value SN65HVD72DR -> THVD1400DR; JLCPCB Part Number C48125 -> C3235232; Manufacturer Part Number SN65HVD72DR -> THVD1400DR
Changed lines of the file:
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@@
 			)
 		)
-		(property "Value" "SN65HVD72DR"
+		(property "Value" "THVD1400DR"
 			(at 173.5933 53.34 0)
 			(show_name no)
@@
 			)
 		)
-		(property "Datasheet" "http://www.ti.com/lit/ds/symlink/sn65hvd11-ht.pdf"
+		(property "Datasheet" "https://www.ti.com/lit/ds/symlink/thvd1400.pdf"
 			(at 171.45 40.64 0)
 			(hide yes)
@@
 			)
 		)
-		(property "Description" "3.3V, RS-485 Transceiver, SOIC-8"
+		(property "Description" "3-5.5V, 500kbps RS-485 Transceiver, SOIC-8"
 			(at 171.45 66.04 0)
 			(hide yes)
@@
 			)
 		)
-		(property "Manufacturer Part Number" "SN65HVD72DR"
+		(property "Manufacturer Part Number" "THVD1400DR"
 			(at 171.45 66.04 0)
 			(hide yes)
@@
 			)
 		)
-		(property "JLCPCB Part Number" "C48125"
+		(property "JLCPCB Part Number" "C3235232"
 			(at 171.45 66.04 0)
 			(hide yes)
