File: Kevin Splitflap/PCBs/power-board/SplitFlapPowerBoard.kicad_sch (KiCad schematic)
At the start: 40 parts, among them J1 KPJX-4S-S, J10 ROCKER SWITCH, J2 ROW 1 (12V B A GND), J3 ROW 2 (12V B A GND), J4 ROW 3 (12V B A GND), J5 GATEWAY PWR (12V GND), J6 GATEWAY RS485 (A B), J7 GATEWAY IO, J8 LED START (12V DIN BIN GND), J9 LED END (12V GND), U1 74AHCT1G125, U2 78L05

Commit message: Power board: jack/switch to the right end, fix DIN jack pinout and position, add rework links
- Mirror the layout left-right: KPJX-4S-S jack and rocker pads at the top-right
  (bottom-left when turned over), wire pads along the bottom edge.
- Jack pinout per Mean Well's R7B plug-face drawing: Kycon pins 2+4 = +12 V,
  1+3 = GND (same side, not diagonal; Mean Well numbers its plug differently).
- Move the jack 4 mm toward the edge so the body face sits on the board edge
  and the 4 mm barrel passes through the panel; fix the footprint outline.
- Jack pin pairs get their own copper, joined to +12V_IN / GND by cuttable
  net-tie links (NT1, NT2) between 16 AWG solder holes, so a reversed plug
  can be fixed with two cuts and two wires. Instructions on the back silk.
- ERC/DRC clean with schematic parity; JLC gerbers, BOM and CPL regenerated.
Parts:
- added NT1, NT2: CUT IF REVERSED, PowerBoard:CutLink_Holes_P6mm, symbol Device:NetTie_2
Connections:
- net +12V_IN: now also NT1.2; no longer J1.1 (Pin_1), J1.4 (Pin_4)
- net GND: now also NT2.2; no longer J1.2 (Pin_2), J1.3 (Pin_3)
- new net JACK_13: J1.1 (Pin_1), J1.3 (Pin_3), NT2.1
- new net JACK_24: J1.2 (Pin_2), J1.4 (Pin_4), NT1.1
